File: H_Bridges/H_Bridges.kicad_pcb (KiCad board)
At the start: 4 copper layers, 112.4 x 81.7 mm, 64 parts, among them J1 S4B-PH-K-SLFSN, J2 USB4085-GF-A_REVB, Q1 IRF540NSTRLPBF, Q10 PMOS, Q2 IRF540NSTRLPBF, Q3 IRF540NSTRLPBF, Q4 IRF540NSTRLPBF, Q5 IRF540NSTRLPBF, Q6 IRF540NSTRLPBF, Q7 IRF540NSTRLPBF, Q8 IRF540NSTRLPBF, Q9 PMOS, U1 ESP8266, U2 max1898eub42+T, U3 TPS61023DRLR

Commit message: made final changes
Parts:
- removed D5: LED, LED_SMD:LED_0402_1005Metric_Pad0.77x0.64mm_HandSolder
- added LED1: 553-0121F, Footprints:553-0121F_DIA, F.Cu at (139.6, 51.3)
- added R17: 300, Resistor_SMD:R_0603_1608Metric, F.Cu at (146.3, 51.4)
- Q10, Q9: value PMOS -> PJC7407_R1_00001
- U1: footprint ESP8266_THT:ESP8266_THT -> Module:Adafruit_HUZZAH_ESP8266_breakout
- moved U1 16.6 mm to (173.4, 104.3)
- moved D4 1.04 mm to (137.2, 81.5)
- moved D7 1.02 mm to (137.3, 83.4)
Routing:
- net Net-(U2-*CHG): track 4.34 -> 43.8 mm, vias 0 -> 1
- net VDD: track 34.6 -> 63.8 mm, vias 0 -> 1
- net Net-(LED1-Pad2): track 0.00 -> 3.36 mm
- net +5V: track 11.2 -> 14.4 mm
- net GND: track 42.0 -> 45.0 mm, vias 27 -> 28
- net /Coil_B+: track 37.1 -> 38.2 mm
- net /Coil_A-: track 35.7 -> 36.8 mm

Commit message: Fab Outputs
Parts:
- moved G*** 0.93 mm to (187.8, 113.6)
Routing:
- net /Charger/VBUS: track 13.0 -> 19.0 mm
Other:
- board text added: "A+ B- A- B+"
- board text added: "AUTO-INJECTION STEPPER MOTOR DRIVER"
- board text added: "MP3"
Changed lines of the file:
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@@
 			(outputformat 1)
 			(mirror no)
-			(drillshape 1)
+			(drillshape 0)
 			(scaleselection 1)
-			(outputdirectory "")
+			(outputdirectory "../Fab/")
 		)
 	)
@@
 	(footprint "LOGO"
 		(layer "F.Cu")
-		(at 187.199908 114.349802 90)
+		(at 187.75 113.6 90)
 		(property "Reference" "G***"
 			(at 0 0 -90)
@@
 		(sheetname "Charger")
 		(sheetfile "chargecircuit.kicad_sch")
-		(attr through_hole)
+		(attr through_hole allow_soldermask_bridges)
 		(fp_line
 			(start 4.47 1.74)
@@
 		(layer "Edge.Cuts")
 	)
+	(gr_text "A+ B- A- B+"
+		(at 166.9 82.35 0)
+		(layer "B.SilkS")
+		(effects
+			(font
+				(size 1 1)
+				(thickness 0.1)
+			)
+			(justify left bottom mirror)
+		)
+	)
+	(gr_text "AUTO-INJECTION\nSTEPPER MOTOR DRIVER\n"
+		(at 190.5 101.9 90)
+		(layer "F.SilkS")
+		(effects
+			(font
+				(size 1 1)
+				(thickness 0.1)
+			)
+			(justify bottom)
+		)
+	)
+	(gr_text "MP3"
+		(at 123 100.8 0)
+		(layer "F.SilkS")
+		(effects
+			(font
+				(size 1 1)
+				(thickness 0.1)
+			)
+			(justify left bottom)
+		)
+	)
 	(segment
 		(start 136.90925 81.54075)
@@
 	)
 	(segment
+		(start 124.375 51.225)
+		(end 124.375 51.83)
+		(width 0.4)
+		(layer "B.Cu")
+		(net 6)
+	)
+	(segment
+		(start 120.125 51.83)
+		(end 120.125 51.275)
+		(width 0.4)
+		(layer "B.Cu")
+		(net 6)
+	)
+	(segment
+		(start 120.125 51.275)
+		(end 120.8 50.6)
+		(width 0.4)
+		(layer "B.Cu")
+		(net 6)
+	)
+	(segment
+		(start 120.8 50.6)
+		(end 123.75 50.6)
+		(width 0.4)
+		(layer "B.Cu")
+		(net 6)
+	)
+	(segment
+		(start 123.75 50.6)
+		(end 124.375 51.225)
+		(width 0.4)
+		(layer "B.Cu")
+		(net 6)
+	)
+	(segment
 		(start 160.77075 69.94075)
 		(end 160.77075 71.27075)
@@
 		(hatch edge 0.5)
 		(connect_pads
-			(clearance 0.5)
+			(clearance 0.3)
 		)
 		(min_thickness 0.25)
 		(filled_areas_thickness no)
 		(fill yes
-			(thermal_gap 0.5)
+			(thermal_gap 0.3)
 			(thermal_bridge_width 0.5)
 		)
@@
 		(polygon
 			(pts
-				(xy 114.85 124.3) (xy 114.85 118.95) (xy 156.85 118.95) (xy 156.85 126.35) (xy 114.85 126.35)
+				(xy 114.85 124.3) (xy 114.85 118.95) (xy 161.7 119) (xy 161.75 127.95) (xy 114.9 127.9)
 			)
 		)
@@
 		(polygon
 			(pts
-				(xy 143.64 51.59) (xy 187.86 51.54) (xy 187.75 110.13) (xy 143.55 110.31)
+				(xy 143.39 48.09) (xy 187.55 47.95) (xy 187.65 110.4) (xy 143.55 110.31)
 			)
 		)
